File: PWM Economizer/PWM Economizer/PWM Economizer.kicad_sch (KiCad schematic)
At the start: 96 parts, among them J1 Conn_01x08_Pin, Q1 PNP, Q2 PNP, U1 DRV103 SO-8, U2 TPS7B8250QDGNRQ1, U3 DRV103 SO-8

Commit message: V1.1 Untested
V1.1 Untested
Parts:
- added D6, D7: D_16V_Zener, Diode_SMD:D_SMB, symbol Device:D_Zener
- added Q3, Q4: SUD50P10-43L, Package_TO_SOT_SMD:TO-252-2, symbol Transistor_FET:SUD50P10-43L
- added R35, R36: 3k, Resistor_SMD:R_0805_2012Metric_Pad1.20x1.40mm_HandSolder, symbol Device:R
- added R37, R38: 100R 2W/3W, SMD_Res_footprints:SMD_Res 3W 12x5.8 & 2512, symbol Resistor_SMD:SMD
- C1, C19, C8: Alt. C1952772 -> C452769 / C167035; LCSC Part C1952730 -> C2798130
- D3: Specs 2-4.5v -> 3.1 - 3.5V (2-4.5v OK)
- J1: now left out of the parts list
- Q1, Q2: Basic Part? E -> B; LCSC Part C516596 -> C8326
- R16, R26: Basic Part? E -> B; LCSC Part C137463 -> C17514
- U1, U3: footprint DRV103:DRV103 PowerPad SOIC Large Heatsink -> DRV103:DRV103 No Heatsink; Alt. (none) -> C1556551; LCSC Part C1556557 -> C1879940; Manufacturer Part No. DRV103H -> DRV103U
Connections:
- net +VDC: now also D6.1 (K), D7.1 (K), Q3.3 (S), Q4.3 (S), R35.2, R36.2; no longer D1.1 (K), D2.1 (K), J1.3 (Pin_3), J1.6 (Pin_6)
- net GND: now also D1.2 (A), D2.2 (A), J1.2 (Pin_2), J1.7 (Pin_7)
- removed net Coil1-: D2.2 (A), J1.2 (Pin_2), U1.5 (OUT)
- removed net Coil2-: D1.2 (A), J1.7 (Pin_7), U3.5 (OUT)
- new net: D7.2 (A), Q4.1 (G), R36.1, R38.1
- new net: D6.2 (A), Q3.1 (G), R35.1, R37.1
- new net: R37.2, U1.5 (OUT)
- new net: R38.2, U3.5 (OUT)
- new net Coil1+: D2.1 (K), J1.3 (Pin_3), Q3.2 (D)
- new net Coil2+: D1.1 (K), J1.6 (Pin_6), Q4.2 (D)
Other:
- note added: "2.3W @ 28v @ Duty Cycle .36W @ 14.2v @ Duty Cycle"
- note added: "Coil1-"
- note added: "Coil2-"
- moved on the sheet: C1, C19, C3, C4
